File: hardware/cursor/PinaBio-v2.0-Cursor/PinaBio-v2.0-Cursor.kicad_sch (KiCad schematic)
At the start: 80 parts, among them J1 USB-C, J2 J_BATT, J3 J_ECG, J4 J_PPG, J5 J_TEMP, J6 J_GSR, J7 J_RESP_T, J8 J_RESP_A, Q1 BSS84, Q2 BSS138, Q3 BSS138, SW1 SW_DPDT, SW2 BOOT, U1 USBLC6-2SC6, U2 BQ24074, U3 TPS63070, U4 TLV75530PDBVR, U5 ESP32-S3-MINI-1U-N8, U6 ADS122C04, U7 ADS122C04, U8 MCP6004

Commit message: Update the Cursor KiCad board to SPEC-0.9
Place the ESP32-S3-MINI-1U U.FL end on the board edge with a copper
keepout, split digital and analogue ground through one wide net tie, and
keep the six electrical changes. ERC and DRC are clean and the fab outputs
are regenerated.
Parts:
- removed U1: USBLC6-2SC6, Package_TO_SOT_SMD:SOT-23-6, symbol Power_Protection:USBLC6-2P6
- added NT1: GND_TIE, PinaCursor:GndTie_2mm, symbol Device:NetTie_2
- added R35, R36: 22, Resistor_SMD:R_0603_1608Metric, symbol Device:R
- added R37: 46.4k 1%, Resistor_SMD:R_0603_1608Metric, symbol Device:R
- added R38: 10k, Resistor_SMD:R_0603_1608Metric, symbol Device:R
- added U1: USBLC6-2SC6, Package_TO_SOT_SMD:SOT-23-6, symbol Power_Protection:USBLC6-2SC6
- C12, C13: footprint Capacitor_SMD:C_0603_1608Metric -> Capacitor_SMD:C_0805_2012Metric
Connections:
- net 3V3_SYS: now also R38.2
- net BOOT: now also R38.1
- net GND: now also NT1.1, R37.2, U1.2 (GND); no longer C18.2, C19.2, C20.2, C21.2, C22.2, J3.2 (Pin_2), J6.2 (Pin_2), J7.2 (Pin_2), J8.2 (Pin_2), R29.2, R34.2, U6.1 (A0), U6.2 (A1), U6.4 (DGND), U6.5 (AVSS), U7.2 (A1), U7.4 (DGND), U7.5 (AVSS), U8.11 (V-)
- net USB_DM: now also R35.1, U1.6 (I/O1); no longer U5.23 (USB_D-)
- net USB_DM_C: now also U1.1 (I/O1)
- net USB_DP: now also R36.1, U1.4 (I/O2); no longer U5.24 (USB_D+)
- net USB_DP_C: now also U1.3 (I/O2)
- net VBUS: now also U1.5 (VBUS)
- net TMR: now reaches U2.14 (TMR)
- net TMR: now also R37.1
- new net AGND: C18.2, C19.2, C20.2, C21.2, C22.2, J3.2 (Pin_2), J6.2 (Pin_2), J7.2 (Pin_2), J8.2 (Pin_2), NT1.2, R29.2, R34.2, U6.1 (A0), U6.2 (A1), U6.4 (DGND), U6.5 (AVSS), U7.2 (A1), U7.4 (DGND), U7.5 (AVSS), U8.11 (V-)
- new net USB_DM_IO: R35.2, U5.23 (USB_D-)
- new net USB_DP_IO: R36.2, U5.24 (USB_D+)
- no-connect marks 29 -> 28
Other:
- note added: "PinaBio v.2.0. Cursor. SPEC-0.9. Sensores sin corte en serie. Interruptor: throw A (pines 1 y 4) es ON. GPIO4=SDA y GPIO5=SCL del bus ADC; GPIO8=SDA y GPIO9=SCL de los modulos. OS del CJMCU-30205 llega a J5 y no tiene GPIO. GPIO0 tiene 10 kΩ a 3V3_SYS. D+/D− llevan 22 Ω entre USBLC6-2SC6 y el ESP32. TMR del BQ24074 lleva 46,4 kΩ a masa. GND y AGND se unen solo en NT1."
- note removed: "PinaBio v.2.0. Cursor. SPEC-0.8. Sensores sin corte en serie. Interruptor: throw A (pines 1 y 4) es ON. GPIO4=SDA y GPIO5=SCL del bus ADC; GPIO8=SDA y GPIO9=SCL de los modulos. OS del CJMCU-30205 llega a J5 y no tiene GPIO."

Commit message: J5 (J_TEMP) pasa a 4 pines: 3V0_TEMP, GND, SDA_MOD, SCL_MOD; se quitan OS y TP1
JST PH B4B-PH-K en esquema, PCB, BOM, position.csv y pinabio.net. A0, A1 y A2 del CJMCU-30205 van a GND en el modulo; OS queda sin conectar. Gerbers, pcb-top.png, ERC y DRC regenerados; spec ES/EN y README actualizados.
Parts:
- removed TP1: OS, TestPoint:TestPoint_Pad_D1.5mm, symbol Connector:TestPoint
- J5: footprint Connector_JST:JST_PH_B8B-PH-K_1x08_P2.00mm_Vertical -> Connector_JST:JST_PH_B4B-PH-K_1x04_P2.00mm_Vertical; symbol Connector_Generic:Conn_01x08 -> Connector_Generic:Conn_01x04
Connections:
- net GND: no longer J5.6 (Pin_6), J5.7 (Pin_7), J5.8 (Pin_8)
- removed net OS: J5.5 (Pin_5)
Other:
- note added: "PinaBio v.2.0. Cursor. SPEC-0.9. Sensores sin corte en serie. Interruptor: throw A (pines 1 y 4) es ON. GPIO4=SDA y GPIO5=SCL del bus ADC; GPIO8=SDA y GPIO9=SCL de los modulos. J5 (J_TEMP) lleva 4 pines: 3V0_TEMP, GND, SDA_MOD, SCL_MOD. A0, A1 y A2 del CJMCU-30205 van a GND en el modulo y OS queda sin conectar. GPIO0 tiene 10 kΩ a 3V3_SYS. D+/D− llevan 22 Ω entre USBLC6-2SC6 y el ESP32. TMR del B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"
- note removed: "PinaBio v.2.0. Cursor. SPEC-0.9. Sensores sin corte en serie. Interruptor: throw A (pines 1 y 4) es ON. GPIO4=SDA y GPIO5=SCL del bus ADC; GPIO8=SDA y GPIO9=SCL de los modulos. OS del CJMCU-30205 llega a J5 y no tiene GPIO. GPIO0 tiene 10 kΩ a 3V3_SYS. D+/D− llevan 22 Ω entre USBLC6-2SC6 y el ESP32. TMR del BQ24074 lleva 46,4 kΩ a masa. GND y AGND se unen solo en NT1."
- moved on the sheet: J6, J7, J8
Changed lines of the file:
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@@
 (instances (project "PinaBio-v2.0-Cursor" (path "/d1bc65b9-079d-45d1-bf50-a5155e2ca362" (reference "J4") (unit 1))))
 )
-(symbol (lib_id "Connector_Generic:Conn_01x08") (at 160.02 106.68 0) (unit 1)
+(symbol (lib_id "Connector_Generic:Conn_01x04") (at 160.02 101.6 0) (unit 1)
 (exclude_from_sim no) (in_bom yes) (on_board yes) (dnp no)
-(property "Reference" "J5" (at 160.02 105.41 0) (effects (font (size 1.27 1.27))))
-(property "Value" "J_TEMP" (at 160.02 109.22 0) (effects (font (size 1.27 1.27))))
-(property "Footprint" "Connector_JST:JST_PH_B8B-PH-K_1x08_P2.00mm_Vertical" (at 160.02 106.68 0) (effects (font (size 1.27 1.27)) (hide yes)))
-(property "Datasheet" "~" (at 160.02 106.68 0) (effects (font (size 1.27 1.27)) (hide yes)))
+(property "Reference" "J5" (at 160.02 100.33 0) (effects (font (size 1.27 1.27))))
+(property "Value" "J_TEMP" (at 160.02 104.14 0) (effects (font (size 1.27 1.27))))
+(property "Footprint" "Connector_JST:JST_PH_B4B-PH-K_1x04_P2.00mm_Vertical" (at 160.02 101.6 0) (effects (font (size 1.27 1.27)) (hide yes)))
+(property "Datasheet" "~" (at 160.02 101.6 0) (effects (font (size 1.27 1.27)) (hide yes)))
 (pin "1")
 (pin "2")
 (pin "3")
 (pin "4")
-(pin "5")
-(pin "6")
-(pin "7")
-(pin "8")
 (instances (project "PinaBio-v2.0-Cursor" (path "/d1bc65b9-079d-45d1-bf50-a5155e2ca362" (reference "J5") (unit 1))))
 )
-(symbol (lib_id "Connector:TestPoint") (at 165.1 99.06 0) (unit 1)
+(symbol (lib_id "Connector_Generic:Conn_01x02") (at 170.18 99.06 0) (unit 1)
 (exclude_from_sim no) (in_bom yes) (on_board yes) (dnp no)
-(property "Reference" "TP1" (at 165.1 97.79 0) (effects (font (size 1.27 1.27))))
-(property "Value" "OS" (at 165.1 101.6 0) (effects (font (size 1.27 1.27))))
-(property "Footprint" "TestPoint:TestPoint_Pad_D1.5mm" (at 165.1 99.06 0) (effects (font (size 1.27 1.27)) (hide yes)))
-(property "Datasheet" "~" (at 165.1 99.06 0) (effects (font (size 1.27 1.27)) (hide yes)))
-(pin "1")
-(instances (project "PinaBio-v2.0-Cursor" (path "/d1bc65b9-079d-45d1-bf50-a5155e2ca362" (reference "TP1") (unit 1))))
+(property "Reference" "J6" (at 170.18 97.79 0) (effects (font (size 1.27 1.27))))
+(property "Value" "J_GSR" (at 170.18 101.6 0) (effects (font (size 1.27 1.27))))
+(property "Footprint" "Connector_JST:JST_PH_B2B-PH-K_1x02_P2.00mm_Vertical" (at 170.18 99.06 0) (effects (font (size 1.27 1.27)) (hide yes)))
+(property "Datasheet" "~" (at 170.18 99.06 0) (effects (font (size 1.27 1.27)) (hide yes)))
+(pin "1")
+(pin "2")
+(instances (project "PinaBio-v2.0-Cursor" (path "/d1bc65b9-079d-45d1-bf50-a5155e2ca362" (reference "J6") (unit 1))))
 )
 (symbol (lib_id "Connector_Generic:Conn_01x02") (at 180.34 99.06 0) (unit 1)
 (exclude_from_sim no) (in_bom yes) (on_board yes) (dnp no)
-(property "Reference" "J6" (at 180.34 97.79 0) (effects (font (size 1.27 1.27))))
-(property "Value" "J_GSR" (at 180.34 101.6 0) (effects (font (size 1.27 1.27))))
+(property "Reference" "J7" (at 180.34 97.79 0) (effects (font (size 1.27 1.27))))
+(property "Value" "J_RESP_T" (at 180.34 101.6 0) (effects (font (size 1.27 1.27))))
 (property "Footprint" "Connector_JST:JST_PH_B2B-PH-K_1x02_P2.00mm_Vertical" (at 180.34 99.06 0) (effects (font (size 1.27 1.27)) (hide yes)))
 (property "Datasheet" "~" (at 180.34 99.06 0) (effects (font (size 1.27 1.27)) (hide yes)))
 (pin "1")
 (pin "2")
-(instances (project "PinaBio-v2.0-Cursor" (path "/d1bc65b9-079d-45d1-bf50-a5155e2ca362" (reference "J6") (unit 1))))
+(instances (project "PinaBio-v2.0-Cursor" (path "/d1bc65b9-079d-45d1-bf50-a5155e2ca362" (reference "J7") (unit 1))))
 )
 (symbol (lib_id "Connector_Generic:Conn_01x02") (at 190.5 99.06 0) (unit 1)
 (exclude_from_sim no) (in_bom yes) (on_board yes) (dnp no)
-(property "Reference" "J7" (at 190.5 97.79 0) (effects (font (size 1.27 1.27))))
-(property "Value" "J_RESP_T" (at 190.5 101.6 0) (effects (font (size 1.27 1.27))))
+(property "Reference" "J8" (at 190.5 97.79 0) (effects (font (size 1.27 1.27))))
+(property "Value" "J_RESP_A" (at 190.5 101.6 0) (effects (font (size 1.27 1.27))))
 (property "Footprint" "Connector_JST:JST_PH_B2B-PH-K_1x02_P2.00mm_Vertical" (at 190.5 99.06 0) (effects (font (size 1.27 1.27)) (hide yes)))
 (property "Datasheet" "~" (at 190.5 99.06 0) (effects (font (size 1.27 1.27)) (hide yes)))
-(pin "1")
-(pin "2")
-(instances (project "PinaBio-v2.0-Cursor" (path "/d1bc65b9-079d-45d1-bf50-a5155e2ca362" (reference "J7") (unit 1))))
-)
-(symbol (lib_id "Connector_Generic:Conn_01x02") (at 200.66 99.06 0) (unit 1)
-(exclude_from_sim no) (in_bom yes) (on_board yes) (dnp no)
-(property "Reference" "J8" (at 200.66 97.79 0) (effects (font (size 1.27 1.27))))
-(property "Value" "J_RESP_A" (at 200.66 101.6 0) (effects (font (size 1.27 1.27))))
-(property "Footprint" "Connector_JST:JST_PH_B2B-PH-K_1x02_P2.00mm_Vertical" (at 200.66 99.06 0) (effects (font (size 1.27 1.27)) (hide yes)))
-(property "Datasheet" "~" (at 200.66 99.06 0) (effects (font (size 1.27 1.27)) (hide yes)))
 (pin "1")
 (pin "2")
@@
 (wire (pts (xy 154.94 104.14) (xy 152.4 104.14)) (stroke (width 0) (type default)))
 (wire (pts (xy 154.94 106.68) (xy 152.4 106.68)) (stroke (width 0) (type default)))
-(wire (pts (xy 154.94 109.22) (xy 152.4 109.22)) (stroke (width 0) (type default)))
-(wire (pts (xy 154.94 111.76) (xy 152.4 111.76)) (stroke (width 0) (type default)))
-(wire (pts (xy 154.94 114.3) (xy 152.4 114.3)) (stroke (width 0) (type default)))
-(wire (pts (xy 154.94 116.84) (xy 152.4 116.84)) (stroke (width 0) (type default)))
-(wire (pts (xy 165.1 99.06) (xy 165.1 101.6)) (stroke (width 0) (type default)))
+(wire (pts (xy 165.1 99.06) (xy 162.56 99.06)) (stroke (width 0) (type default)))
+(wire (pts (xy 165.1 101.6) (xy 162.56 101.6)) (stroke (width 0) (type default)))
 (wire (pts (xy 175.26 99.06) (xy 172.72 99.06)) (stroke (width 0) (type default)))
 (wire (pts (xy 175.26 101.6) (xy 172.72 101.6)) (stroke (width 0) (type default)))
 (wire (pts (xy 185.42 99.06) (xy 182.88 99.06)) (stroke (width 0) (type default)))
 (wire (pts (xy 185.42 101.6) (xy 182.88 101.6)) (stroke (width 0) (type default)))
-(wire (pts (xy 195.58 99.06) (xy 193.04 99.06)) (stroke (width 0) (type default)))
-(wire (pts (xy 195.58 101.6) (xy 193.04 101.6)) (stroke (width 0) (type default)))
 (label "GND" (at 27.94 68.58 90) (effects (font (size 1.27 1.27)) (justify left bottom)))
 (label "GND" (at 35.56 68.58 90) (effects (font (size 1.27 1.27)) (justify left bottom)))
@@
 (label "SDA_MOD" (at 152.4 104.14 180) (effects (font (size 1.27 1.27)) (justify left bottom)))
 (label "SCL_MOD" (at 152.4 106.68 180) (effects (font (size 1.27 1.27)) (justify left bottom)))
-(label "OS" (at 152.4 109.22 180) (effects (font (size 1.27 1.27)) (justify left bottom)))
-(label "GND" (at 152.4 111.76 180) (effects (font (size 1.27 1.27)) (justify left bottom)))
-(label "GND" (at 152.4 114.3 180) (effects (font (size 1.27 1.27)) (justify left bottom)))
-(label "GND" (at 152.4 116.84 180) (effects (font (size 1.27 1.27)) (justify left bottom)))
-(label "OS" (at 165.1 101.6 90) (effects (font (size 1.27 1.27)) (justify left bottom)))
-(label "SNS_GSR" (at 172.72 99.06 180) (effects (font (size 1.27 1.27)) (justify left bottom)))
+(label "SNS_GSR" (at 162.56 99.06 180) (effects (font (size 1.27 1.27)) (justify left bottom)))
+(label "AGND" (at 162.56 101.6 180) (effects (font (size 1.27 1.27)) (justify left bottom)))
+(label "SNS_TH" (at 172.72 99.06 180) (effects (font (size 1.27 1.27)) (justify left bottom)))
 (label "AGND" (at 172.72 101.6 180) (effects (font (size 1.27 1.27)) (justify left bottom)))
-(label "SNS_TH" (at 182.88 99.06 180) (effects (font (size 1.27 1.27)) (justify left bottom)))
+(label "SNS_AB" (at 182.88 99.06 180) (effects (font (size 1.27 1.27)) (justify left bottom)))
 (label "AGND" (at 182.88 101.6 180) (effects (font (size 1.27 1.27)) (justify left bottom)))
-(label "SNS_AB" (at 193.04 99.06 180) (effects (font (size 1.27 1.27)) (justify left bottom)))
-(label "AGND" (at 193.04 101.6 180) (effects (font (size 1.27 1.27)) (justify left bottom)))
 (no_connect (at 50.8 55.88))
 (no_connect (at 50.8 58.42))
@@
 (no_connect (at 711.2 81.28))
 (no_connect (at 711.2 83.82))
-(text "PinaBio v.2.0. Cursor. SPEC-0.9. Sensores sin corte en serie. Interruptor: throw A (pines 1 y 4) es ON. GPIO4=SDA y GPIO5=SCL del bus ADC; GPIO8=SDA y GPIO9=SCL de los modulos. OS del CJMCU-30205 llega a J5 y no tiene GPIO. GPIO0 tiene 10 kΩ a 3V3_SYS. D+/D− llevan 22 Ω entre USBLC6-2SC6 y el ESP32. TMR del BQ24074 lleva 46,4 kΩ a masa. GND y AGND se unen solo en NT1." (at 25.4 12.7 0) (effects (font (size 2.0 2.0))))
+(text "PinaBio v.2.0. Cursor. SPEC-0.9. Sensores sin corte en serie. Interruptor: throw A (pines 1 y 4) es ON. GPIO4=SDA y GPIO5=SCL del bus ADC; GPIO8=SDA y GPIO9=SCL de los modulos. J5 (J_TEMP) lleva 4 pines: 3V0_TEMP, GND, SDA_MOD, SCL_MOD. A0, A1 y A2 del CJMCU-30205 van a GND en el modulo y OS queda sin conectar. GPIO0 tiene 10 kΩ a 3V3_SYS. D+/D− llevan 22 Ω entre USBLC6-2SC6 y el ESP32. TMR del BQ24074 lleva 46,4 kΩ a masa. GND y AGND se unen solo en NT1." (at 25.4 12.7 0) (effects (font (size 2.0 2.0))))
 (sheet_instances (path "/" (page "1")))
 (embedded_fonts no)

Commit message: Add purchasable BOM fields and schematic-PCB parity
Symbols and bom.csv now carry manufacturer and MPN, and capacitors
carry voltage and dielectric. Footprints keep the library nickname and
unconnected pads use the schematic net name. Electrical values, tracks
and copper are unchanged.
Parts:
- C1: Dielectric (none) -> X5R; MPN (none) -> CL10A475KO8NNNC; Manufacturer (none) -> Samsung Electro-Mechanics; Voltage (none) -> 16V
- C10, C16, C2, C3, C4, C5, C6: Dielectric (none) -> X5R; MPN (none) -> CL21A106KOQNNNE; Manufacturer (none) -> Samsung Electro-Mechanics; Voltage (none) -> 16V
- C11, C14, C17, C18, C19, C20, C21, C22: Dielectric (none) -> X7R; MPN (none) -> CL10B104KB8NNNC; Manufacturer (none) -> Samsung Electro-Mechanics; Voltage (none) -> 50V
- C12, C13: Dielectric (none) -> X7R; MPN (none) -> CL21B225KAFNNNE; Manufacturer (none) -> Samsung Electro-Mechanics; Voltage (none) -> 25V
- C15: Dielectric (none) -> X5R; MPN (none) -> CL10A105KB8NNNC; Manufacturer (none) -> Samsung Electro-Mechanics; Voltage (none) -> 50V
- C7, C8, C9: Dielectric (none) -> X5R; MPN (none) -> CL21A226MAYNNNE; Manufacturer (none) -> Samsung Electro-Mechanics; Voltage (none) -> 25V
- D1: MPN (none) -> BZX84-C3V6,215; Manufacturer (none) -> Nexperia
- J1: MPN (none) -> HC-TYPE-C-16P-01A; Manufacturer (none) -> HCTL
- J2: MPN (none) -> B3B-PH-K-S(LF)(SN); Manufacturer (none) -> JST
- J3: MPN (none) -> B6B-PH-K-S(LF)(SN); Manufacturer (none) -> JST
- J4: MPN (none) -> B5B-PH-K-S(LF)(SN); Manufacturer (none) -> JST
- J5: MPN (none) -> B4B-PH-K-S(LF)(SN); Manufacturer (none) -> JST
- J6, J7, J8: MPN (none) -> B2B-PH-K-S(LF)(SN); Manufacturer (none) -> JST
- Q1: MPN (none) -> BSS84LT1G; Manufacturer (none) -> onsemi
- Q2, Q3: MPN (none) -> BSS138LT1G; Manufacturer (none) -> onsemi
- R1, R2: MPN (none) -> RC0603FR-075K1L; Manufacturer (none) -> YAGEO
- R10, R11, R12, R19, R20, R21, R30, R31, R32, R9: MPN (none) -> RC0603FR-07100KL; Manufacturer (none) -> YAGEO
- R13: MPN (none) -> RT0603BRD0749K9L; Manufacturer (none) -> YAGEO
- R14: MPN (none) -> RT0603BRD0716KL; Manufacturer (none) -> YAGEO
- R15, R3: MPN (none) -> RC0603JR-070RL; Manufacturer (none) -> YAGEO
- R16, R17: MPN (none) -> RC0603FR-071ML; Manufacturer (none) -> YAGEO
- R18: MPN (none) -> RC0603FR-07330KL; Manufacturer (none) -> YAGEO
- R22, R25, R26, R27, R29, R38, R4: MPN (none) -> RC0603FR-0710KL; Manufacturer (none) -> YAGEO
- R23, R24: MPN (none) -> RC0603FR-074K7L; Manufacturer (none) -> YAGEO
- R28: MPN (none) -> RC0603FR-0756KL; Manufacturer (none) -> YAGEO
- R33: MPN (none) -> RC0603FR-0733K2L; Manufacturer (none) -> YAGEO
- R34: MPN (none) -> RC0603FR-0747K5L; Manufacturer (none) -> YAGEO
- R35, R36: MPN (none) -> RC0603FR-0722RL; Manufacturer (none) -> YAGEO
- R37: MPN (none) -> RC0603FR-0746K4L; Manufacturer (none) -> YAGEO
- R5: MPN (none) -> RC0603FR-0715KL; Manufacturer (none) -> YAGEO
- R6, R7: MPN (none) -> RC0603FR-072K94L; Manufacturer (none) -> YAGEO
- R8: MPN (none) -> RC0603FR-072K2L; Manufacturer (none) -> YAGEO
- SW1: MPN (none) -> JS202011JCQN; Manufacturer (none) -> C&K
- SW2: MPN (none) -> B3U-1000P; Manufacturer (none) -> Omron
- U1: MPN (none) -> USBLC6-2SC6; Manufacturer (none) -> STMicroelectronics
- U2: MPN (none) -> BQ24074RGTR; Manufacturer (none) -> Texas Instruments
- U3: MPN (none) -> TPS63070RNMR; Manufacturer (none) -> Texas Instruments
- U4: MPN (none) -> TLV75530PDBVR; Manufacturer (none) -> Texas Instruments
- U5: MPN (none) -> ESP32-S3-MINI-1U-N8; Manufacturer (none) -> Espressif
- U6, U7: MPN (none) -> ADS122C04IPWR; Manufacturer (none) -> Texas Instruments
- U8: MPN (none) -> MCP6004-I/SL; Manufacturer (none) -> Microchip

Commit message: Dejar el DPDT en la caja y fijar la bobina XAL4020
Seis taladros conservan las redes del interruptor, con ON, OFF y COM en la serigrafía. La pieza de caja es el C&K 7201SYZQE. L1 queda como Coilcraft XAL4020-152ME. La masa del TPS63070 no se mueve.
Parts:
- L1: MPN (none) -> XAL4020-152ME; Manufacturer (none) -> Coilcraft
- SW1: value SW_DPDT -> DPDT caja; footprint Button_Switch_SMD:SW_DPDT_CK_JS202011JCQN -> PinaCursor:SW_ext_6pad; MPN JS202011JCQN -> (none); Manufacturer C&K -> (none)
Other:
- note added: "PinaBio v.2.0. Cursor. SPEC-0.9. Sensores sin corte en serie. Interruptor de caja C&K 7201SYZQE, DPDT ON-ON, cable 1:1. ON (lejos de la chaveta) cierra 2-1 y 5-4: EN2_CE a VLOG y TPS_EN a BAT_PROT. OFF (hacia la chaveta) cierra 2-3 y 5-6: EN2_CE a GND y TPS_EN a VLOG. Comunes en terminales 2 y 5. L1 es Coilcraft XAL4020-152ME, 1,5 uH. GPIO4=SDA y GPIO5=SCL del bus ADC; GPIO8=SDA y GPIO9=SCL de lo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"
- note removed: "PinaBio v.2.0. Cursor. SPEC-0.9. Sensores sin corte en serie. Interruptor: throw A (pines 1 y 4) es ON. GPIO4=SDA y GPIO5=SCL del bus ADC; GPIO8=SDA y GPIO9=SCL de los modulos. J5 (J_TEMP) lleva 4 pines: 3V0_TEMP, GND, SDA_MOD, SCL_MOD. A0, A1 y A2 del CJMCU-30205 van a GND en el modulo y OS queda sin conectar. GPIO0 tiene 10 kΩ a 3V3_SYS. D+/D− llevan 22 Ω entre USBLC6-2SC6 y el ESP32. TMR del B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"
