File: hardware/PinaBio-v2.0-ChatGPT/PinaBio-v2.0-ChatGPT.kicad_pcb (KiCad board)
At the start: 4 copper layers, 84.5 x 53.1 mm, 89 parts, among them J1 USB-C, J2 J_BATT, J3 J_ECG, J4 J_PPG, J5 J_TEMP, J6 J_GSR, J7 J_RESP_T, J8 J_RESP_A, J9 J_BATT_METER, Q1 BSS84, Q2 BSS138, Q3 BSS138, Q4 BSS84, Q5 BSS138, SW1 DPDT caja, SW2 BOOT, U1 USBLC6-2SC6, U2 BQ24074, U3 TPS63070, U4 TLV75530PDBVR, U5 ESP32-S3-MINI-1U-N8, U6 ADS122C04, U7 ADS122C04, U8 MCP6004

Commit message: Refine ChatGPT board silkscreen and fabrication outputs
Other:
- board text added: ""Paca" v.2.0."
- board text added: "BATT"
- board text added: "PINABio"
- board text added: "VIN"
- board text removed: "BATERIA"
- board text removed: "PinaBio Paca v.2.0."
