File: hardware/PinaBio-v2.0-ChatGPT/PinaBio-v2.0-ChatGPT.kicad_sch (KiCad schematic)
At the start: 93 parts, among them J1 USB-C USB2.0 16P, J2 LiPo 1S protected + NTC, J3 AD8232 external module, J4 GSR, J5 RESP_T, J6 RESP_A, J7 GY-30102 external, J8 CJMCU-30205 external, J9 DEBUG UART, SW1 ON/OFF DPDT, SW2 BOOT, SW3 RESET, U1 USBLC6-2SC6, U2 BQ24074RGT, U3 TPS63070RNM, U4 TLV75530PDBVR, U5 ESP32-S3-MINI-1U-N8, U6 ADS122C04IPW, U7 ADS122C04IPW, U8 MCP6004

Commit message: Complete PinaBio Paca v2 ChatGPT KiCad 9 prototype
Parts:
- removed C23: 100nF X7R, Capacitor_SMD:C_0603_1608Metric, symbol Device:C
- removed C24, C25, C26: 1uF X7R, Capacitor_SMD:C_0603_1608Metric, symbol Device:C
- removed D1: BZT52C3V3, Diode_SMD:D_SOD-123, symbol Device:D_Zener
- removed D2: SMF5.0A, Diode_SMD:D_SOD-123F, symbol Device:D_TVS
- removed J4: GSR, Connector_PinHeader_2.54mm:PinHeader_1x02_P2.54mm_Vertical, symbol Connector_Generic:Conn_01x02
- removed J5: RESP_T, Connector_PinHeader_2.54mm:PinHeader_1x02_P2.54mm_Vertical, symbol Connector_Generic:Conn_01x02
- removed J7: GY-30102 external, Connector_PinHeader_2.54mm:PinHeader_1x05_P2.54mm_Vertical, symbol Connector_Generic:Conn_01x05
- removed J8: CJMCU-30205 external, Connector_PinHeader_2.54mm:PinHeader_1x08_P2.54mm_Vertical, symbol Connector_Generic:Conn_01x08
- removed J9: DEBUG UART, Connector_PinHeader_2.54mm:PinHeader_1x04_P2.54mm_Vertical, symbol Connector_Generic:Conn_01x04
- removed R41, R42: 4.7k, Resistor_SMD:R_0603_1608Metric, symbol Device:R
- removed R43, R44: 10k, Resistor_SMD:R_0603_1608Metric, symbol Device:R
- removed SW1: ON/OFF DPDT, Button_Switch_SMD:SW_DPDT_CK_JS202011JCQN, symbol Switch:SW_DPDT_x2
- removed SW3: RESET, Button_Switch_SMD:SW_SPST_TL3305A, symbol Switch:SW_Push
- removed U3: TPS63070RNM, PinaBio-ChatGPT:TPS63070_RNM0015A, symbol PinaBio:TPS63070RNM
- removed U4: TLV75530PDBVR, Package_TO_SOT_SMD:SOT-23-5, symbol PinaBio:TLV75530PDBV
- removed U5: ESP32-S3-MINI-1U-N8, PinaBio-ChatGPT:ESP32-S3-MINI-1U, symbol RF_Module:ESP32-S3-MINI-1U
- removed U6, U7: ADS122C04IPW, Package_SO:TSSOP-16_4.4x5mm_P0.65mm, symbol PinaBio:ADS122C04IPW
- removed U8: MCP6004, Package_SO:SOIC-14_3.9x8.7mm_P1.27mm, symbol PinaBio:MCP6004
- added D1: BZX84-C3V6, Package_TO_SOT_SMD:SOT-23, symbol Diode:BZX84Cxx
- added J4: J_PPG, Connector_JST:JST_PH_B5B-PH-K_1x05_P2.00mm_Vertical, symbol Connector_Generic:Conn_01x05
- added J5: J_TEMP, Connector_JST:JST_PH_B4B-PH-K_1x04_P2.00mm_Vertical, symbol Connector_Generic:Conn_01x04
- added J7: J_RESP_T, Connector_JST:JST_PH_B2B-PH-K_1x02_P2.00mm_Vertical, symbol Connector_Generic:Conn_01x02
- added J8: J_RESP_A, Connector_JST:JST_PH_B2B-PH-K_1x02_P2.00mm_Vertical, symbol Connector_Generic:Conn_01x02
- added J9: J_BATT_METER, Connector_JST:JST_PH_B2B-PH-K_1x02_P2.00mm_Vertical, symbol Connector_Generic:Conn_01x02
- added NT1: GND_TIE, PinaCursor:GndTie_2mm, symbol Device:NetTie_2
- added Q1, Q4: BSS84, Package_TO_SOT_SMD:SOT-23, symbol Transistor_FET:TP0610T
- added Q2, Q3, Q5: BSS138, Package_TO_SOT_SMD:SOT-23, symbol Transistor_FET:Q_NMOS_GSD
- added SW1: DPDT caja, PinaCursor:SW_ext_6pad, symbol Switch:SW_Slide_DPDT
- added U3: TPS63070, PinaCursor:TPS63070RNM, symbol PinaCursor:TPS63070
- added U4: TLV75530PDBVR, Package_TO_SOT_SMD:SOT-23-5, symbol Regulator_Linear:TLV70012_SOT23-5
- added U5: ESP32-S3-MINI-1U-N8, RF_Module:ESP32-S2-MINI-1U, symbol RF_Module:ESP32-S3-MINI-1
- added U6, U7: ADS122C04, Package_SO:TSSOP-16_4.4x5mm_P0.65mm, symbol PinaCursor:ADS122C04PW
- added U8: MCP6004, Package_SO:SOIC-14_3.9x8.7mm_P1.27mm, symbol Amplifier_Operational:LM2902
- C1: value 1uF 16V X7R -> 4.7uF; Dielectric (none) -> X5R; MPN (none) -> CL10A475KO8NNNC; Manufacturer (none) -> Samsung Electro-Mechanics; Voltage (none) -> 16V
- C10: value 2.2uF 6.3V X7R -> 10uF; Dielectric (none) -> X5R; MPN (none) -> CL21A106KOQNNNE; Manufacturer (none) -> Samsung Electro-Mechanics; Voltage (none) -> 16V
- C11: value 2.2uF 6.3V X7R -> 100nF; footprint Capacitor_SMD:C_0805_2012Metric -> Capacitor_SMD:C_0603_1608Metric; Dielectric (none) -> X7R; MPN (none) -> CL10B104KB8NNNC; Manufacturer (none) -> Samsung Electro-Mechanics; Voltage (none) -> 50V
- C12: value 1uF X7R -> 2.2uF; footprint Capacitor_SMD:C_0603_1608Metric -> Capacitor_SMD:C_0805_2012Metric; Dielectric (none) -> X7R; MPN (none) -> CL21B225KAFNNNE; Manufacturer (none) -> Samsung Electro-Mechanics; Voltage (none) -> 25V
- C13: value 100nF X7R -> 2.2uF; footprint Capacitor_SMD:C_0603_1608Metric -> Capacitor_SMD:C_0805_2012Metric; Dielectric (none) -> X7R; MPN (none) -> CL21B225KAFNNNE; Manufacturer (none) -> Samsung Electro-Mechanics; Voltage (none) -> 25V
- C14: value 10uF 6.3V X7R -> 100nF; footprint Capacitor_SMD:C_0805_2012Metric -> Capacitor_SMD:C_0603_1608Metric; Dielectric (none) -> X7R; MPN (none) -> CL10B104KB8NNNC; Manufacturer (none) -> Samsung Electro-Mechanics; Voltage (none) -> 50V
- C15: value 100nF X7R -> 1uF; Dielectric (none) -> X5R; MPN (none) -> CL10A105KB8NNNC; Manufacturer (none) -> Samsung Electro-Mechanics; Voltage (none) -> 50V
- C16: value 10uF 6.3V X7R -> 10uF; Dielectric (none) -> X5R; MPN (none) -> CL21A106KOQNNNE; Manufacturer (none) -> Samsung Electro-Mechanics; Voltage (none) -> 16V
- C17, C18, C19, C20: value 100nF X7R -> 100nF; Dielectric (none) -> X7R; MPN (none) -> CL10B104KB8NNNC; Manufacturer (none) -> Samsung Electro-Mechanics; Voltage (none) -> 50V
- C2: value 4.7uF 10V X7R -> 10uF; footprint Capacitor_SMD:C_0603_1608Metric -> Capacitor_SMD:C_0805_2012Metric; Dielectric (none) -> X5R; MPN (none) -> CL21A106KOQNNNE; Manufacturer (none) -> Samsung Electro-Mechanics; Voltage (none) -> 16V
- C21: value 33nF X7R -> 100nF; Dielectric (none) -> X7R; MPN (none) -> CL10B104KB8NNNC; Manufacturer (none) -> Samsung Electro-Mechanics; Voltage (none) -> 50V
- C22: value 1uF X7R -> 100nF; Dielectric (none) -> X7R; MPN (none) -> CL10B104KB8NNNC; Manufacturer (none) -> Samsung Electro-Mechanics; Voltage (none) -> 50V
- C3, C4, C5: value 10uF 10V X7R -> 10uF; footprint Capacitor_SMD:C_0603_1608Metric -> Capacitor_SMD:C_0805_2012Metric; Dielectric (none) -> X5R; MPN (none) -> CL21A106KOQNNNE; Manufacturer (none) -> Samsung Electro-Mechanics; Voltage (none) -> 16V
- C6: value 100nF X7R -> 10uF; footprint Capacitor_SMD:C_0603_1608Metric -> Capacitor_SMD:C_0805_2012Metric; Dielectric (none) -> X5R; MPN (none) -> CL21A106KOQNNNE; Manufacturer (none) -> Samsung Electro-Mechanics; Voltage (none) -> 16V
- C7, C8, C9: value 22uF 6.3V X7R -> 22uF; Dielectric (none) -> X5R; MPN (none) -> CL21A226MAYNNNE; Manufacturer (none) -> Samsung Electro-Mechanics; Voltage (none) -> 25V
- J1: value USB-C USB2.0 16P -> USB-C; footprint Connector_USB:USB_C_Receptacle_HRO_TYPE-C-31-M-12 -> Connector_USB:USB_C_Receptacle_HCTL_HC-TYPE-C-16P-01A; MPN (none) -> HC-TYPE-C-16P-01A; Manufacturer (none) -> HCTL
- J2: value LiPo 1S protected + NTC -> J_BATT; footprint Connector_JST:JST_PH_S3B-PH-K_1x03_P2.00mm_Horizontal -> Connector_JST:JST_PH_B3B-PH-K_1x03_P2.00mm_Vertical; MPN (none) -> B3B-PH-K-S(LF)(SN); Manufacturer (none) -> JST
- J3: value AD8232 external module -> J_ECG; footprint Connector_PinHeader_2.54mm:PinHeader_1x06_P2.54mm_Vertical -> Connector_JST:JST_PH_B6B-PH-K_1x06_P2.00mm_Vertical; MPN (none) -> B6B-PH-K-S(LF)(SN); Manufacturer (none) -> JST
- J6: value RESP_A -> J_GSR; footprint Connector_PinHeader_2.54mm:PinHeader_1x02_P2.54mm_Vertical -> Connector_JST:JST_PH_B2B-PH-K_1x02_P2.00mm_Vertical; MPN (none) -> B2B-PH-K-S(LF)(SN); Manufacturer (none) -> JST
- L1: value XAL4020-152MEC 1.5uH -> 1.5uH; MPN (none) -> XAL4020-152MEC; Manufacturer (none) -> Coilcraft
- R1, R2: value 5.1k 1% -> 5.1k; MPN (none) -> RC0603FR-075K1L; Manufacturer (none) -> YAGEO
- R10: value 46.4k 1% -> 100k; MPN (none) -> RC0603FR-07100KL; Manufacturer (none) -> YAGEO
- R11, R12: value 10k -> 100k; MPN (none) -> RC0603FR-07100KL; Manufacturer (none) -> YAGEO
- R13: MPN (none) -> RT0603BRD0749K9L; Manufacturer (none) -> YAGEO
- R14: MPN (none) -> RT0603BRD0716KL; Manufacturer (none) -> YAGEO
- R15: value 10k -> 0; MPN (none) -> RC0603JR-070RL; Manufacturer (none) -> YAGEO
- R16: value 0R -> 1M; MPN (none) -> RC0603FR-071ML; Manufacturer (none) -> YAGEO
- R17: value 10k -> 1M; MPN (none) -> RC0603FR-071ML; Manufacturer (none) -> YAGEO
- R18: value 10k -> 330k; MPN (none) -> RC0603FR-07330KL; Manufacturer (none) -> YAGEO
- R19: value 1M 1% -> 100k; MPN (none) -> RC0603FR-07100KL; Manufacturer (none) -> YAGEO
- R20: value 330k 1% -> 100k; MPN (none) -> RC0603FR-07100KL; Manufacturer (none) -> YAGEO
- R21: MPN (none) -> RC0603FR-07100KL; Manufacturer (none) -> YAGEO
- R22: value 100k -> 10k; MPN (none) -> RC0603FR-0710KL; Manufacturer (none) -> YAGEO
- R23: value 100k -> 4.7k; MPN (none) -> RC0603FR-074K7L; Manufacturer (none) -> YAGEO
- R24: value 2.2k -> 4.7k; MPN (none) -> RC0603FR-074K7L; Manufacturer (none) -> YAGEO
- R25: value 2.2k -> 10k; MPN (none) -> RC0603FR-0710KL; Manufacturer (none) -> YAGEO
- R26, R27, R39: MPN (none) -> RC0603FR-0710KL; Manufacturer (none) -> YAGEO
- R28: value 33.2k 1% -> 56k 1%; MPN (none) -> RC0603FR-0756KL; Manufacturer (none) -> YAGEO
- R29: value 47.5k 1% -> 10k 1%; MPN (none) -> RC0603FR-0710KL; Manufacturer (none) -> YAGEO
- R3: value 100k 1% -> 0; MPN (none) -> RC0603JR-070RL; Manufacturer (none) -> YAGEO
- R30: value 56k 1% -> 100k; MPN (none) -> RC0603FR-07100KL; Manufacturer (none) -> YAGEO
- R31: value 10k 1% -> 100k; MPN (none) -> RC0603FR-07100KL; Manufacturer (none) -> YAGEO
- R32: value 100k 1% -> 100k; MPN (none) -> RC0603FR-07100KL; Manufacturer (none) -> YAGEO
- R33: value 100k 1% -> 33.2k 1%; MPN (none) -> RC0603FR-0733K2L; Manufacturer (none) -> YAGEO
- R34: value 100k 1% -> 47.5k 1%; MPN (none) -> RC0603FR-0747K5L; Manufacturer (none) -> YAGEO
- R35, R36: value 100k 1% -> 22; MPN (none) -> RC0603FR-0722RL; Manufacturer (none) -> YAGEO
- R37: value 100k 1% -> 46.4k 1%; MPN (none) -> RC0603FR-0746K4L; Manufacturer (none) -> YAGEO
- R38: value 10k 1% -> 10k; MPN (none) -> RC0603FR-0710KL; Manufacturer (none) -> YAGEO
- R4: value 150k 1% -> 10.0k; MPN (none) -> RC0603FR-0710KL; Manufacturer (none) -> YAGEO
- R40: value 10k 1% -> 1M; MPN (none) -> RC0603FR-071ML; Manufacturer (none) -> YAGEO
- R5: value 22R -> 15.0k; MPN (none) -> RC0603FR-0715KL; Manufacturer (none) -> YAGEO
- R6: value 22R -> 2.94k 1%; MPN (none) -> RC0603FR-072K94L; Manufacturer (none) -> YAGEO
- R7: value 3.00k 1% -> 2.94k 1%; MPN (none) -> RC0603FR-072K94L; Manufacturer (none) -> YAGEO
- R8: value 3.00k 1% -> 2.2k; MPN (none) -> RC0603FR-072K2L; Manufacturer (none) -> YAGEO
- R9: value 1.50k 1% -> 100k; MPN (none) -> RC0603FR-07100KL; Manufacturer (none) -> YAGEO
- SW2: footprint Button_Switch_SMD:SW_SPST_TL3305A -> Button_Switch_SMD:SW_SPST_B3U-1000P; MPN (none) -> B3U-1000P; Manufacturer (none) -> Omron
- U1: MPN (none) -> USBLC6-2SC6; Manufacturer (none) -> STMicroelectronics
- U2: value BQ24074RGT -> BQ24074; MPN (none) -> BQ24074RGTR; Manufacturer (none) -> Texas Instruments
Connections:
- net ADC_DRDY_ECG is gone; now on net 3V3_SYS: R26.2
- net ADC_DRDY_SLOW is gone; now on net 3V3_SYS: R27.2
- net ADC_SCL is gone; now on net 3V3_SYS: R25.2
- net ADC_SDA is gone; now on net 3V3_SYS: R24.2
- net BQ_MODE_SENSE is gone; now on net 3V3_SYS: R21.2
- net ECG_SDN is gone; now on net 3V3_A: J3.6 (Pin_6)
- net GSR_ADC is gone; now on net 3V3_SYS: R38.2
- net GSR_BUF is gone; now on net BOOT: R38.1
- net RESP_A_ADC is gone; now on net BAT_PROT: R40.2
- net RESP_A_SENSE is gone; now on net GND: R37.2
- net RESP_T_BUF is gone; now on net TPS_EN: R39.1
- net TPS_PG is gone; now on net 3V3_A: R15.2
- net TPS_VAUX is gone; now on net SYS: C6.1
- net USB_DN_MCU is gone; now on net GND: R5.2
- net USB_DP_MCU is gone; now on net GND: R6.2
- net 0V5_EXC: now also R30.1, R31.1, U8.1, U8.2 (-); no longer R33.1, R34.1
- net 3V0_TEMP: now also C13.1, J5.1 (Pin_1), U4.5 (OUT); no longer C11.1
- net 3V3_A: now also C22.1, J3.2 (Pin_2), R28.1, U6.10 (AIN1), U6.12 (AVDD), U6.6 (AIN3), U6.7 (AIN2), U6.8 (REFN), U6.9 (REFP), U7.12 (AVDD), U7.6 (AIN3), U7.8 (REFN), U7.9 (REFP), U8.4 (V+); no longer J3.1 (Pin_1), R16.2, R30.1
- net 3V3_SYS: now also C12.1, C21.1, R10.2, R19.1, R22.2, R23.2, R9.2, J4.1 (Pin_1), Q2.1 (G), Q5.1 (G), U3.7 (VOUT), U3.8 (VOUT), U4.1 (IN), U4.3 (EN), U5.3 (3V3), U6.13 (DVDD), U6.3 (RESET), U7.1 (A0), U7.13 (DVDD), U7.3 (RESET); no longer C14.1, C15.1, R11.1, R12.1, R16.1, R17.1, R18.1, R24.1, R25.1, R26.1, R27.1
- net BAT_PROT: now also C3.1, R16.2, Q1.2 (S), Q4.2 (S), SW1.4 (A); no longer C2.1, R19.1
- net BAT_SENSE: now also C14.1, R17.2, R18.1, U5.5 (IO1); no longer C13.1, R19.2, R20.1
- net ECG_OUT: now also R33.1; no longer R28.1
- net GND: now also R11.2, R12.2, R18.2, R19.2, D1.1 (A), J4.2 (Pin_2), J5.2 (Pin_2), J9.2 (Pin_2), NT1.1, Q2.2 (S), Q3.2 (S), Q5.2 (S), SW1.3 (C), U3.1 (PS/SYNC), U3.10 (PGND), U3.15 (VSEL), U3.4 (GND), U3.6 (FB2), U4.2 (GND), U5.1 (GND), U5.2 (GND), U5.42 (GND), U5.43 (GND), U5.46 (GND), U5.47 (GND), U5.48 (GND), U5.49 (GND), U5.50 (GND), U5.51 (GND), U5.52 (GND), U5.53 (GND), U5.54 (GND), U5.55 (GND), U5.56 (GND), U5.57 (GND), U5.58 (GND), U5.59 (GND), U5.60 (GND), U5.61 (GND), U5.62 (GND), U5.63 (GND), U5.64 (GND), U5.65 (GND); no longer C18.2, C19.2, C20.2, C21.2, C22.2, J3.2 (Pin_2), J6.2 (Pin_2), R10.2, R20.2, R23.2, R29.2, R31.2, R4.2, R9.2
- net PPG_INT: now also R25.1, J4.5 (Pin_5), U5.14 (IO10)
- net SYS: now also C2.1, U3.12 (VIN), U3.13 (VIN); no longer C3.1
- net TPS_EN: now also R12.1, SW1.5 (B); no longer R22.1
- net VBUS_RAW: now also R3.2; no longer J1.A4 (VBUS), J1.A9 (VBUS), J1.B4 (VBUS), J1.B9 (VBUS), R3.1, U1.5 (VBUS)
- net BAT_NTC renamed TS
- net BOOT_IO0 renamed BOOT
- net BOOT: now also U5.4 (IO0); no longer R18.2
- net BQ_CHG renamed CHG
- net CHG: now also R9.1; no longer R12.2
- net BQ_EN2_CE renamed EN2_CE
- net EN2_CE: now also R11.1, SW1.2 (B); no longer R21.1
- net BQ_ILIM renamed ILIM
- net ILIM: now also R8.1; no longer R9.1
- net BQ_ISET renamed ISET
- net ISET: now also R6.1; no longer R7.1
- net BQ_ITERM renamed ITERM
- net ITERM: now also R7.1; no longer R8.1
- net BQ_TMR renamed PGOOD
- net PGOOD: now also U2.7 (~{PGOOD}); no longer U2.14 (TMR)
- net ECG_ADC renamed DIV_EXC
- net DIV_EXC: now also U8.3 (+); no longer C21.1
- net ECG_LON renamed LO_P
- net LO_P: now also U5.15 (IO11)
- net ECG_LOP renamed LO_N
- net LO_N: now also U5.16 (IO12)
- removed net ESP_EN: C12.1, R17.2
- removed net EXC_DIV: C22.1, R30.2, R31.1
- net GSR_ELECTRODE renamed SNS_AB
- net SNS_AB: now also J8.1 (Pin_1), U8.12 (+); no longer R35.1
- net GSR_SENSE renamed USB_DM_IO
- net USB_DM_IO: now also U5.23 (USB_D-)
- net RESP_A_BUF renamed METER_GATE
- net METER_GATE: now also Q4.1 (G), Q5.3 (D)
- removed net RESP_A_ELECTRODE: J6.1 (Pin_1), R34.2, R37.1
- net RESP_T_ADC renamed TPS_EN_IC
- net TPS_EN_IC: now also U3.14 (EN)
- net RESP_T_ELECTRODE renamed ECG_DIV
- net ECG_DIV: now also R34.1, U6.11 (AIN0); no longer R36.1
- net RESP_T_SENSE renamed USB_DP_IO
- net USB_DP_IO: now also U5.24 (USB_D+)
- net SW_ON_SENSE renamed SDA_ADC
- net SDA_ADC: now also U5.8 (IO4), U6.15 (SDA), U7.15 (SDA); no longer R22.2
- net TPS_FB renamed FB
- net FB: now also U3.5 (FB)
- net TPS_L1 renamed SW_L1
- net SW_L1: now also U3.11 (L1)
- net TPS_L2 renamed SW_L2
- net SW_L2: now also U3.9 (L2)
- net USB_DN_ESD renamed USB_DM
- net USB_DM: now also R35.1; no longer R5.1
- net USB_DN_RAW renamed USB_DM_C
- net USB_DP_ESD renamed USB_DP
- net USB_DP: now also R36.1; no longer R6.1
- net USB_DP_RAW renamed USB_DP_C
- removed net USB_VALID_N: R11.2, U2.7 (~{PGOOD})
- removed net VBUS_MODE: R3.2, R4.1, U2.6 (EN1)
- new net AGND: C18.2, C19.2, C20.2, C21.2, C22.2, J3.1 (Pin_1), J6.2 (Pin_2), J7.2 (Pin_2), J8.2 (Pin_2), NT1.2, R29.2, R34.2, U6.1 (A0), U6.2 (A1), U6.4 (DGND), U6.5 (AVSS), U7.2 (A1), U7.4 (DGND), U7.5 (AVSS), U8.11 (V-)
- new net BAT_METER: J9.1 (Pin_1), Q4.3 (D)
- new net DIV_IN: Q1.3 (D), R17.1
- new net DRDY_ECG: R26.1, U5.10 (IO6), U6.14 (DRDY)
- new net DRDY_SLOW: R27.1, U5.11 (IO7), U7.14 (DRDY)
- new net EN_MOD: C15.1, R22.1, U5.45 (EN)
- new net OUT_AB: U7.7 (AIN2), U8.13 (-), U8.14
- new net OUT_GSR: U7.11 (AIN0), U8.6 (-), U8.7
- new net OUT_TH: U7.10 (AIN1), U8.8, U8.9 (-)
- new net Q1G: Q1.1 (G), Q2.3 (D), R16.1
- new net SCL_ADC: R24.1, U5.9 (IO5), U6.16 (SCL), U7.16 (SCL)
- new net SCL_MOD: J4.3 (Pin_3), J5.4 (Pin_4), U5.13 (IO9)
- new net SDA_MOD: J4.4 (Pin_4), J5.3 (Pin_3), U5.12 (IO8)
- new net SNS_GSR: J6.1 (Pin_1), R30.2, U8.5 (+)
- new net SNS_TH: J7.1 (Pin_1), R31.2, U8.10 (+)
- new net TMR: R37.1, U2.14 (TMR)
- new net VAUX: C11.1, U3.3 (VAUX)
- new net VBUS: J1.A4 (VBUS), J1.A9 (VBUS), J1.B4 (VBUS), J1.B9 (VBUS), R3.1, R4.1, U1.5 (VBUS)
- new net VBUS_G: Q3.1 (G), R20.2
- new net VBUS_N: Q3.3 (D), R21.1, U5.6 (IO2)
- new net VLOG: D1.3 (K), R20.1, R4.2, R5.1, SW1.1 (A), SW1.6 (C), U2.6 (EN1)
- no-connect marks 30 -> 28
Other:
- note added: "PinaBio v.2.0. Cursor. SPEC-0.9. Sensores sin corte en serie. Interruptor de caja C&K 7201SYZQE, DPDT ON-ON, cable 1:1. ON (lejos de la chaveta) cierra 2-1 y 5-4: EN2_CE a VLOG y TPS_EN a BAT_PROT. OFF (hacia la chaveta) cierra 2-3 y 5-6: EN2_CE a GND y TPS_EN a VLOG. Comunes en terminales 2 y 5. L1 es Coilcraft XAL4020-152MEC, 1,5 uH. GPIO4=SDA y GPIO5=SCL del bus ADC; GPIO8=SDA y GPIO9=SCL de l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"
- note removed: "1 USB-C, bateria y cargador"
- note removed: "2 Reguladores y conmutacion ON/OFF"
- note removed: "3 ESP32-S3 y control"
- note removed: "4 ADC, ECG y sensores externos"
- note removed: "5 GSR, bandas y acondicionamiento"
- note removed: "Conectores de sensores permanentemente cableados: no hay relés ni cortes automáticos."
- note removed: "ON + USB: batería alimenta; no carga; aislador externo obligatorio con persona. OFF + USB: carga/programación, sin persona."
- note removed: "REVISIÓN DE INGENIERÍA — comprobar módulos, potencia, pruebas sobre cuerpo y huellas antes de fabricar"
- company: PINA - Experimental biofeedback -> (none)
- title: PinaBio v2.0 ChatGPT -> PinaBio v.2.0. Cursor
